File: PCB/DifferentialProbe/DifferentialProbe.kicad_pcb (KiCad board)
At the start: 2 copper layers, 56.5 x 100 mm, 33 parts, among them U1 IFNU411, U2 HFA3046BZ

Commit message: 1st design finished
Parts:
- added C15: 22pF, Capacitor_THT:C_Disc_D3.0mm_W1.6mm_P2.50mm, F.Cu at (35.1, -61.2)
- added C17: 68pF, Capacitor_THT:C_Disc_D3.0mm_W1.6mm_P2.50mm, F.Cu at (32.7, -61.2)
- added C18: 33pF, Capacitor_THT:C_Disc_D3.0mm_W1.6mm_P2.50mm, F.Cu at (42.8, -44.5)
- added C20: 100nF, Capacitor_THT:C_Disc_D4.3mm_W1.9mm_P5.00mm, F.Cu at (8.76, -51.0)
- added C21: 100nF, Capacitor_THT:C_Disc_D4.3mm_W1.9mm_P5.00mm, F.Cu at (10.7, -47.9)
- added C22: 10nF, Capacitor_THT:C_Disc_D3.0mm_W1.6mm_P2.50mm, F.Cu at (35.2, -75.0)
- added C23: 6p8F, Capacitor_THT:C_Disc_D3.0mm_W1.6mm_P2.50mm, F.Cu at (47.6, -54.4)
- added C24: 6p8F, Capacitor_THT:C_Disc_D3.0mm_W1.6mm_P2.50mm, F.Cu at (32.5, -68.1)
- added C25: 100nF, Capacitor_THT:C_Disc_D4.3mm_W1.9mm_P5.00mm, F.Cu at (55.2, -64.1)
- added C26: 100nF, Capacitor_THT:C_Disc_D4.3mm_W1.9mm_P5.00mm, F.Cu at (52.6, -52.1)
- added C39: Not Fitted, Capacitor_THT:C_Disc_D4.3mm_W1.9mm_P5.00mm, F.Cu at (55.1, -44.9)
- added D3: LED, LED_THT:LED_D3.0mm, F.Cu at (11.4, -53.0)
- added J1: Scope Signal, Connector_Wire:SolderWire-2.5sqmm_1x01_D2.4mm_OD4.4mm, F.Cu at (40.4, -36.6)
- added J2: Scope Ground / Screen, Connector_Wire:SolderWire-2.5sqmm_1x01_D2.4mm_OD4.4mm, F.Cu at (27.6, -36.6)
- added J3: Wire A, BVKSound:Wire_Hole, F.Cu at (37.3, -81.5)
- added J4: Wire B, BVKSound:Wire_Hole, F.Cu at (19.3, -81.3)
- added J5: Wire A, BVKSound:Wire_Hole, F.Cu at (8.64, -66.8)
- added J6: Wire B, BVKSound:Wire_Hole, F.Cu at (5.84, -66.8)
- added J7: Wire +9V, BVKSound:Wire_Hole, F.Cu at (27.8, -77.0)
- added J8: Wire +9V, BVKSound:Wire_Hole, F.Cu at (55.1, -64.8)
- added Q1: 2N2222A, Package_TO_SOT_THT:TO-18-3, F.Cu at (12.6, -58.6)
- added Q2: 2N2907A, Package_TO_SOT_THT:TO-18-3, F.Cu at (2.77, -53.6)
- added R10: 374R, Resistor_THT:R_Axial_DIN0207_L6.3mm_D2.5mm_P10.16mm_Horizontal, F.Cu at (40.1, -46.4)
- added R11: 18K, Resistor_THT:R_Axial_DIN0204_L3.6mm_D1.6mm_P7.62mm_Horizontal, F.Cu at (42.8, -49.1)
- added R12: 2K2, Resistor_THT:R_Axial_DIN0207_L6.3mm_D2.5mm_P10.16mm_Horizontal, F.Cu at (27.1, -54.6)
- added R13: 2K2, Resistor_THT:R_Axial_DIN0207_L6.3mm_D2.5mm_P10.16mm_Horizontal, F.Cu at (29.7, -56.6)
- added R15: 210R, Resistor_THT:R_Axial_DIN0207_L6.3mm_D2.5mm_P10.16mm_Horizontal, F.Cu at (23.5, -64.8)
- added R17: 210R, Resistor_THT:R_Axial_DIN0207_L6.3mm_D2.5mm_P2.54mm_Vertical, F.Cu at (14.2, -65.4)
- added R18: 620R, Resistor_THT:R_Axial_DIN0207_L6.3mm_D2.5mm_P2.54mm_Vertical, F.Cu at (2.45, -48.1)
- added R19: 6K8, Resistor_THT:R_Axial_DIN0207_L6.3mm_D2.5mm_P10.16mm_Horizontal, F.Cu at (5.55, -45.0)
- added R20: 510R, Resistor_THT:R_Axial_DIN0204_L3.6mm_D1.6mm_P7.62mm_Horizontal, F.Cu at (40.7, -75.0)
- added R21: 4K42, Resistor_THT:R_Axial_DIN0207_L6.3mm_D2.5mm_P10.16mm_Horizontal, F.Cu at (45.0, -47.9)
- added R22: 4K42, Resistor_THT:R_Axial_DIN0207_L6.3mm_D2.5mm_P10.16mm_Horizontal, F.Cu at (28.5, -70.8)
- added R7: 7R5, Resistor_THT:R_Axial_DIN0204_L3.6mm_D1.6mm_P7.62mm_Horizontal, F.Cu at (55.0, -52.0)
- added R8: 3K48, Resistor_THT:R_Axial_DIN0207_L6.3mm_D2.5mm_P10.16mm_Horizontal, F.Cu at (24.0, -44.5)
- added R9: 4K02, Resistor_THT:R_Axial_DIN0207_L6.3mm_D2.5mm_P10.16mm_Horizontal, F.Cu at (20.5, -64.8)
- added RV2: 1K, BVKSound:67WR10KLF, F.Cu at (19.6, -46.2)
- added RV3: 500R, BVKSound:3362P_1, F.Cu at (40.2, -58.1)
- added RV4: 100K, BVKSound:64W_1, F.Cu at (48.9, -71.6)
- added SW1: Attenuation Switch, BVKSound:SSSF011700, F.Cu at (33.6, -48.4)
- added U3: AD797, Package_DIP:DIP-8_W7.62mm, F.Cu at (45.1, -64.7)
- R16: footprint Resistor_THT:R_Axial_DIN0204_L3.6mm_D1.6mm_P2.54mm_Vertical -> Resistor_THT:R_Axial_DIN0207_L6.3mm_D2.5mm_P2.54mm_Vertical
- moved C2 86.9 mm to (48.0, -78.9), turned to 45 degrees
- moved C7 83.1 mm to (32.6, -90.0)
- moved C9 82.8 mm to (32.6, -85.8)
- moved RV1 74.1 mm to (27.1, -85.5), turned to 90 degrees
- moved D1 72.7 mm to (8.57, -66.5), turned to 90 degrees
- moved D2 72.3 mm to (5.79, -66.5), turned to 90 degrees
- moved C8 70.1 mm to (32.6, -87.9)
- moved C16 67.7 mm to (3.01, -65.0), turned to 90 degrees
- moved C11 67.0 mm to (21.6, -90.0)
- moved C3 67.0 mm to (39.5, -81.0), turned to 350 degrees
- moved U2 63.7 mm to (23.4, -59.9), turned to 90 degrees
- moved C12 59.9 mm to (21.6, -87.9)
- moved R2a1 57.8 mm to (41.4, -87.3), turned to 340 degrees
- moved C14 54.4 mm to (22.9, -79.5), turned to 180 degrees
- moved C13 53.3 mm to (21.6, -85.8)
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- renumbered C15 to C19
Connections:
- U1 pad 1: Net-(U1-Pad1) -> Net-(RV2-Pad1)
- U2 pad 1: Net-(U2-Pad1) -> Net-(Q1-Pad1)
- U2 pad 11: Net-(U2-Pad11) -> Net-(R16-Pad2)
- U2 pad 12: Net-(U2-Pad12) -> Net-(Q1-Pad1)
- U2 pad 13: Net-(U2-Pad13) -> -9V
- U2 pad 14: Net-(U2-Pad14) -> Net-(Q1-Pad1)
- U2 pad 2: Net-(U2-Pad2) -> Net-(Q1-Pad1)
- U2 pad 3: Net-(U2-Pad3) -> -9V
- U2 pad 4: Net-(U2-Pad12) -> Net-(Q1-Pad1)
- U2 pad 6: Net-(U2-Pad6) -> Net-(RV2-Pad1)
- U2 pad 8: Net-(U2-Pad8) -> Net-(R14-Pad2)
Routing:
- net GND: track 0.00 -> 203.8 mm, vias 0 -> 5
- net -9V: track 0.00 -> 130.7 mm, vias 0 -> 2
- net Net-(C22-Pad2): track 0.00 -> 50.6 mm, vias 0 -> 1
- net Net-(C15-Pad2): track 0.00 -> 49.9 mm
- net Net-(RV2-Pad1): track 0.00 -> 43.9 mm, vias 0 -> 1
- net Net-(R17-Pad2): track 0.00 -> 39.5 mm, vias 0 -> 2
- net Net-(C10-Pad1): track 0.00 -> 31.7 mm
- net Net-(R14-Pad2): track 0.00 -> 31.3 mm
- net +9V: track 0.00 -> 31.1 mm
- net Net-(C39-Pad1): track 0.00 -> 29.0 mm
- net Net-(C15-Pad1): track 0.00 -> 27.1 mm
- net Net-(R16-Pad2): track 0.00 -> 26.8 mm, vias 0 -> 1
- net Net-(C11-Pad1): track 0.00 -> 26.7 mm
- net Net-(Q1-Pad1): track 0.00 -> 25.9 mm, vias 0 -> 2
- net Net-(C20-Pad2): track 0.00 -> 25.9 mm
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- added copper zone on B.Cu, net GND
- added copper zone on F.Cu, net GND
Other:
- outline, holes or cut-outs redrawn
- board text added: "Input+"
- board text added: "Input-"

Commit message: finalized rev0 for ordering
Other:
- board text added: "BVKSound Differential Probe 2021 Rev0"
